File: KiCad/5 Step Sequencer.kicad_sch (KiCad schematic)
At the start: 65 parts, among them J1 RESET IN, J2 TRIG IN, J4 CV OUT, J5 TRIG OUT, Q2 BC856, SW1 SW_SPDT_321, SW2 SW_SPDT_321, SW3 SW_SPDT_321, SW4 SW_SPDT_321, SW5 SW_SPDT_321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

Commit message: routing
Parts:
- added TP1: A, TestPoint:TestPoint_Pad_D1.5mm, symbol Connector:TestPoint
- added TP10: F, TestPoint:TestPoint_Pad_D1.5mm, symbol Connector:TestPoint
- added TP11, TP12: GND, TestPoint:TestPoint_Pad_D1.5mm, symbol Connector:TestPoint
- added TP2: B, TestPoint:TestPoint_Pad_D1.5mm, symbol Connector:TestPoint
- added TP3: C, TestPoint:TestPoint_Pad_D1.5mm, symbol Connector:TestPoint
- added TP8: D, TestPoint:TestPoint_Pad_D1.5mm, symbol Connector:TestPoint
- added TP9: E, TestPoint:TestPoint_Pad_D1.5mm, symbol Connector:TestPoint
Connections:
- net +5V: now also TP10.1
- net GND: now also TP11.1, TP12.1
- net RESET IN: now also TP1.1
- net TEMPO: now also TP8.1
- net TRIGGER IN: now also TP2.1
- net at C1.1, D5.1 (K), D6.1 (K)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: now also TP9.1
- net at D10.2 (A), D11.2 (A), D12.2 (A)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: now also TP3.1

Commit message: adding new logo, troubleshooting, gerber
Other:
- company: Dirty Dream - Nathanael Noir -> © Dirty Dream - Nathanael Noir
- title: 5 Step Sequencer -> Pentastable Sequencer
