File: KiCad/power.kicad_sch (KiCad schematic)
At the start: 17 parts, among them J3 Connector Header, U1 TL072

Commit message: adding new logo, troubleshooting, gerber
Other:
- company: Dirty Dream - Nathanael Noir -> © Dirty Dream - Nathanael Noir
- title: 5 Step Sequencer -> Pentastable Sequencer
Changed lines of the file:
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@@
 	(paper "A4")
 	(title_block
-		(title "5 Step Sequencer")
-		(date "2026-03-13")
+		(title "Pentastable Sequencer")
+		(date "2026-04-02")
 		(rev "v1.0")
-		(company "Dirty Dream - Nathanael Noir")
+		(company "© Dirty Dream - Nathanael Noir")
 		(comment 1 "A 5 step sequencer inspired by the Buchla Sound Easel")
 	)
